Commit message: gnss fixes

File: tuna_description/urdf/boat.urdf (robot description, URDF)
Before this commit: robot ros_car, 3 links, 2 joints
Joints:
- joint base_to_gps: origin xyz=0.016 0 0.12 rpy=0 0 0 -> xyz=0.016 0 0.12 rpy=0 0 -1.5708

Commit message: safety light widget, fixed odom map publisher

File: tuna_description/urdf/boat.urdf (robot description, URDF)
Before this commit: robot ros_car, 3 links, 2 joints
Joints:
- joint base_to_gps: origin xyz=0.016 0 0.12 rpy=0 0 -1.5708 -> xyz=0.016 0 0.12 rpy=0 0 0

Commit message: urdf update

File: tuna_description/urdf/boat.urdf (robot description, URDF)
Before this commit: robot ros_car, 3 links, 2 joints
Links:
- added link prop_left; visual mesh filename=package://tuna_description/meshes/prop_left.dae
- added link prop_right; visual mesh filename=package://tuna_description/meshes/prop_right.dae
Joints:
- added joint base_to_prop_left: type continuous, parent base_link, child prop_left, origin xyz=-0.14 0.018 -0.043 rpy=0 -0.19 0, axis 1 0 0, limit effort=1 velocity=12
- added joint base_to_prop_right: type continuous, parent base_link, child prop_right, origin xyz=-0.14 -0.018 -0.043 rpy=0 -0.19 0, axis 1 0 0, limit effort=1 velocity=12

Commit message: moved meshes, add gazebo world

File: tuna_description/urdf/boat.urdf (robot description, URDF)
Before this commit: robot tuna, 5 links, 4 joints
Links:
- link base_link: geometry visual mesh filename=package://tuna_gazebo/meshes/boat.dae
- link prop_left: geometry visual mesh filename=package://tuna_gazebo/meshes/prop_left.dae
- link prop_right: geometry visual mesh filename=package://tuna_gazebo/meshes/prop_right.dae
